File: mannuino.kicad_sch (KiCad schematic)
At the start: 27 parts, among them J1 USB_C_Receptacle_USB2.0_16P, J2 Conn_01x13, J3 Conn_01x15, J4 Conn_01x15, SW1 SW_Push, SW2 SW_Push, U1 ESP32-S3-MINI-1U, U2 USBLC6-2SC6, U3 XC6220B331MR

Commit message: COMMIT
Parts:
- U1: footprint RF_Module:ESP32-S2-MINI-1U -> RF_Module:ESP32-S3-WROOM-1U
Changed lines of the file:
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@@
 			)
 		)
-		(property "Footprint" "RF_Module:ESP32-S2-MINI-1U"
+		(property "Footprint" "RF_Module:ESP32-S3-WROOM-1U"
 			(at 187.96 22.86 0)
 			(effects

Commit message: :heavysob:
Parts:
- removed C1: 1uF, 10V(20%), Capacitor_SMD:C_0805_2012Metric, symbol Device:C
- removed D1: SK6812MINI, LED_SMD:LED_SK6812MINI_PLCC4_3.5x3.5mm_P1.75mm, symbol LED:SK6812MINI
- removed R1: 10k, Resistor_SMD:R_0603_1608Metric, symbol Device:R
- removed U1: ESP32-S3-MINI-1U, RF_Module:ESP32-S3-WROOM-1U, symbol RF_Module:ESP32-S3-MINI-1U
- added U4: ESP32-S3-WROOM-2, RF_Module:ESP32-S3-WROOM-1U, symbol RF_Module:ESP32-S3-WROOM-2
Connections:
- net GPIO31 is gone; now on net GND: J2.11 (Pin_11)
- net GPIO32 is gone; now on net GND: J2.12 (Pin_12)
- net GPIO33 is gone; now on net GND: J2.13 (Pin_13)
- net +3V3: now also J2.8 (Pin_8), J2.9 (Pin_9), U4.2 (3V3); no longer J2.5 (Pin_5)
- net +5V: now also J2.5 (Pin_5)
- net GND: now also U4.1 (GND), U4.40 (GND), U4.41 (GND); no longer J2.8 (Pin_8), J2.9 (Pin_9)
- net GPIO0: now also U4.39 (IO1)
- net GPIO1: now also U4.38 (IO2)
- net GPIO11: now also U4.19 (IO11)
- net GPIO12: now also U4.20 (IO12)
- net GPIO13: now also U4.21 (IO13)
- net GPIO14: now also U4.22 (IO14)
- net GPIO15: now also U4.8 (IO15)
- net GPIO16: now also U4.9 (IO16)
- net GPIO17: now also U4.10 (IO17)
- net GPIO18: now also U4.11 (IO18)
- net GPIO19: now also U4.23 (IO21)
- net GPIO2: now also U4.15 (IO3)
- net GPIO20: now also U4.31 (IO38)
- net GPIO21: now also U4.32 (MTCK/IO39)
- net GPIO22: now also U4.33 (MTDO/IO40)
- net GPIO23: now also U4.34 (MTDI/IO41)
- net GPIO24: now also U4.35 (MTMS/IO42)
- net GPIO25: now also U4.37 (TXD0/IO43)
- net GPIO26: now also U4.36 (RXD0/IO44)
- net GPIO27: now also U4.26 (IO45)
- net GPIO28: now also U4.16 (IO46)
- net GPIO29: now also U4.24 (IO47)
- net GPIO3: now also U4.4 (IO4)
- net GPIO30: now also U4.25 (IO48)
- net GPIO4: now also U4.5 (IO5)
- net GPIO5: now also U4.6 (IO6)
- net GPIO6: now also U4.7 (IO7)
- net GPIO7: now also U4.12 (IO8)
- net GPIO8: now also U4.17 (IO9)
- net GPIO9: now also U4.18 (IO10)
- net USB_D+: now also U4.14 (USB_D+/IO20)
- net USB_D-: now also U4.13 (USB_D-/IO19)
- net boot: now also U4.27 (IO0)
- net en: now also U4.3 (EN)
- no-connect marks 5 -> 2
Other:
- note removed: "Led"
- moved on the sheet: C8, C9

Commit message: IG last version
Parts:
- removed J2: Conn_01x13, Connector_PinHeader_2.00mm:PinHeader_1x13_P2.00mm_Vertical, symbol Connector_Generic:Conn_01x13
- removed J3, J4: Conn_01x15, Connector_PinHeader_2.00mm:PinHeader_1x15_P2.00mm_Vertical, symbol Connector_Generic:Conn_01x15
- added J2, J3: Conn_01x20, Connector_PinHeader_2.00mm:PinHeader_1x20_P2.00mm_Vertical, symbol Connector_Generic:Conn_01x20
Connections:
- net +3V3: now also J2.18 (Pin_18), J3.18 (Pin_18)
- net +5V: now also J2.19 (Pin_19), J2.2 (Pin_2), J3.19 (Pin_19), J3.2 (Pin_2)
- net GND: now also J2.1 (Pin_1), J2.20 (Pin_20), J3.1 (Pin_1), J3.20 (Pin_20)
- net GPIO0: now also J2.3 (Pin_3)
- net GPIO1: now also J2.4 (Pin_4)
- net GPIO11: now also J3.13 (Pin_13)
- net GPIO12: now also J3.14 (Pin_14)
- net GPIO13: now also J3.15 (Pin_15)
- net GPIO14: now also J2.5 (Pin_5)
- net GPIO15: now also J3.17 (Pin_17)
- net GPIO16: now also J3.3 (Pin_3)
- net GPIO17: now also J3.4 (Pin_4)
- net GPIO18: now also J3.16 (Pin_16)
- net GPIO19: now also J2.6 (Pin_6)
- net GPIO2: now also J3.5 (Pin_5)
- net GPIO20: now also J2.12 (Pin_12)
- net GPIO21: now also J2.11 (Pin_11)
- net GPIO22: now also J2.10 (Pin_10)
- net GPIO23: now also J2.9 (Pin_9)
- net GPIO24: now also J2.8 (Pin_8)
- net GPIO25: now also J2.7 (Pin_7)
- net GPIO26: now also J2.13 (Pin_13)
- net GPIO27: now also J2.14 (Pin_14)
- net GPIO28: now also J2.15 (Pin_15)
- net GPIO29: now also J2.16 (Pin_16)
- net GPIO3: now also J3.6 (Pin_6)
- net GPIO30: now also J2.17 (Pin_17)
- net GPIO4: now also J3.7 (Pin_7)
- net GPIO5: now also J3.8 (Pin_8)
- net GPIO6: now also J3.9 (Pin_9)
- net GPIO7: now also J3.10 (Pin_10)
- net GPIO8: now also J3.11 (Pin_11)
- net GPIO9: now also J3.12 (Pin_12)
