File: pcb/mannuino.kicad_pcb (KiCad board)
At the start: 2 copper layers, 34 x 41.3 mm, 23 parts, among them J1 USB_C_Receptacle_USB2.0_16P, J2 Conn_01x20, J3 Conn_01x20, SW1 SW_Push, SW2 SW_Push, U2 USBLC6-2SC6, U3 XC6220B331MR, U4 ESP32-S3-WROOM-2

Commit message: Fix a few things with the pcb
Routing:
- net /boot: track 38.8 -> 34.8 mm
- net /GPIO18: track 24.2 -> 22.6 mm
- net /GPIO19: track 30.5 -> 28.9 mm
- net GND: track 83.3 -> 81.9 mm, vias 27 -> 24
- net +5V: track 115.9 -> 115.0 mm
- net /GPIO14: track 39.7 -> 39.1 mm
